Commit message: added camera plugin and launch files

File: src/arduinobot_description/urdf/arduino-bot.urdf.xacro (robot description, xacro)
@@ -6,7 +6,7 @@
     <xacro:arg name="is_sim" default="true"/>
     <!-- Include Gazebo Parameters -->
-    <!-- <xacro:include filename="$(find arduino_bot_description)/urdf/arduinobot_gazebo.xacro" /> -->
+    <xacro:include filename="$(find arduinobot_description)/urdf/arduinobot_gazebo.xacro" />
     <!-- Include ros2_control Plugins -->
-    <!-- <xacro:include filename="$(find arduino_bot_description)/urdf/arduinobot_ros2_control.xacro" /> -->
+    <!-- <xacro:include filename="$(find arduinobot_description)/urdf/arduinobot_ros2_control.xacro" /> -->
   <xacro:property name="PI" value="3.14159265359"/>
   <xacro:property name="effort" value="30.0"/>
@@ -128,4 +128,5 @@
   </link>
   <link name="rgb_camera">
+      <xacro:default_inertial mass="0.001"/>
       <visual>
             <origin rpy="-1.57 0 -1.57" xyz="-0.1 0.125 0.15"/>
@@ -134,10 +135,10 @@
             </geometry>
       </visual>
-      <collisison>
+      <collision>
             <origin rpy="-1.57 0 -1.57" xyz="-0.1 0.125 0.15"/>
             <geometry>
                 <mesh filename="package://arduinobot_description/meshes/pi_camera.STL" scale="0.01 0.01 0.01"/>
             </geometry>
-      </collisison>
+      </collision>
   </link>
   <joint name="virtual_joint" type="fixed">

File: src/arduinobot_description/urdf/arduinobot_gazebo.xacro (robot description, xacro)
@@ -1,18 +1,32 @@
 <?xml version="1.0"?>
 <robot xmlns:xacro="http://www.ros.org/wiki/xacro" name="arduinobot">
+  <!---->
   <!-- ROS 2 Control -->
-  <gazebo>
-    <!-- ROS 2 Humble -->
-    <xacro:if value="$(arg is_ignition)">
-      <plugin filename="ign_ros2_control-system" name="ign_ros2_control::IgnitionROS2ControlPlugin">
-        <parameters>$(find arduinobot_controller)/config/arduinobot_controllers.yaml</parameters>
-      </plugin>
-    </xacro:if>
-    <!-- ROS 2 Iron or above -->
-    <xacro:unless value="$(arg is_ignition)">
-      <plugin filename="gz_ros2_control-system" name="gz_ros2_control::GazeboSimROS2ControlPlugin">
-        <parameters>$(find arduinobot_controller)/config/arduinobot_controllers.yaml</parameters>
-      </plugin>
-    </xacro:unless>
+<gazebo reference="rgb_camera">
+  <sensor type="camera" name="camera">
+    <always_on>true</always_on>
+    <update_rate>30</update_rate>
+    <visualize>true</visualize>
+    <camera>
+      <horizontal_fov>1.15</horizontal_fov>
+      <image>
+        <width>2304</width>
+        <height>1296</height>
+        <format>R8G8B8</format>
+      </image>
+      <clip>
+        <near>0.1</near>
+        <far>100</far>
+      </clip>
+    </camera>
+    <plugin name="gazebo_ros_camera" filename="libgazebo_ros_camera.so">
+      <ros>
+        <remapping>image_raw:=image_raw</remapping>
+        <remapping>camera_info:=camera_info</remapping>
+      </ros>
+      <camera_name>camera</camera_name>
+      <frame_name>/rgb_camera</frame_name>
+    </plugin>
+  </sensor>
 </gazebo>
 </robot>

Commit message: corrected the control setup for hardware

File: src/arduinobot_description/urdf/arduino-bot.urdf.xacro (robot description, xacro)
@@ -8,5 +8,5 @@
     <xacro:include filename="$(find arduinobot_description)/urdf/arduinobot_gazebo.xacro" />
     <!-- Include ros2_control Plugins -->
-    <!-- <xacro:include filename="$(find arduinobot_description)/urdf/arduinobot_ros2_control.xacro" /> -->
+    <xacro:include filename="$(find arduinobot_description)/urdf/arduinobot_ros2_control.xacro" />
   <xacro:property name="PI" value="3.14159265359"/>
   <xacro:property name="effort" value="30.0"/>

File: src/arduinobot_description/urdf/arduino_ros2_control.xacro (robot description, xacro)
@@ -17,8 +17,4 @@
                 </hardware>
             </xacro:unless>
-            <joint name="joint_6">
-                <param name="mimic">joint_5</param>
-                <param name="multiplier">-1</param>
-            </joint>
         </xacro:if>
         <!-- ros2_control Real Robot -->
@@ -57,4 +53,8 @@
             <state_interface name="position"/>
         </joint>
+        <joint name="joint_6">
+                <param name="mimic">joint_5</param>
+                <param name="multiplier">-1</param>
+        </joint>
     </ros2_control>
 </robot>

File: src/arduinobot_description/urdf/arduinobot_gazebo.xacro (robot description, xacro)
@@ -3,4 +3,18 @@
   <!---->
   <!-- ROS 2 Control -->
+<gazebo>
+    <!-- ROS 2 Humble -->
+    <xacro:if value="$(arg is_ignition)">
+      <plugin filename="ign_ros2_control-system" name="ign_ros2_control::IgnitionROS2ControlPlugin">
+        <parameters>$(find arduinobot_controller)/config/arduinobot_controllers.yaml</parameters>
+      </plugin>
+    </xacro:if>
+    <!-- ROS 2 Iron or above -->
+    <xacro:unless value="$(arg is_ignition)">
+      <plugin filename="gz_ros2_control-system" name="gz_ros2_control::GazeboSimROS2ControlPlugin">
+        <parameters>$(find arduinobot_controller)/config/arduinobot_controllers.yaml</parameters>
+      </plugin>
+    </xacro:unless>
+</gazebo>
 <gazebo reference="rgb_camera">
   <sensor type="camera" name="camera">

Commit message: implemted control and its launch file

File: src/arduinobot_description/urdf/arduino-bot.urdf.xacro (robot description, xacro)
@@ -186,5 +186,5 @@
     <child link="gripper_left"/>
     <limit lower="0.0" upper="${PI/2}" effort="${effort}" velocity="${velocity}"/>
-    <minic joint="joint_5" multiplier="-1"/>
+    <mimic joint="joint_5" multiplier="-1"/>
   </joint>
   <joint name ="rgb_camera_joint" type="fixed">

File: src/arduinobot_description/urdf/arduino_ros2_control.xacro (robot description, xacro)
@@ -8,5 +8,5 @@
             <xacro:if value="$(arg is_ignition)">
                 <hardware>
-                    <plugin>ign_ros2_control/IgnitionSystem</plugin>
+                    <plugin>mock_components/GenericSystem</plugin>
                 </hardware>
             </xacro:if>
